File: Hardware/2021_Rev1/2021_Rev2.sch (KiCad schematic (older format))
At the start: 39 parts, among them J1 USB_A, U1 TM4C129E_Launchpad, U2 OKI, U3 OKI, U4 FT230XS

Commit message: Rev2 Update
Swapped the ctl pins to  usable ones and removed usb/keyboard functionality and 5v regular for usb
Parts:
- removed 100nF1: C_Small, Capacitor_SMD:C_0603_1608Metric_Pad1.08x0.95mm_HandSolder, symbol Device:C_Small
- removed 4.7uF1: C_Polarized_Small_US, Capacitor_THT:CP_Radial_D5.0mm_P2.50mm, symbol Device:C_Polarized_Small_US
- removed C3, C4: 10uF, Capacitor_SMD:C_0603_1608Metric_Pad1.08x0.95mm_HandSolder, symbol Device:C_Small
- removed C7: 100nF, Capacitor_SMD:C_0603_1608Metric_Pad1.08x0.95mm_HandSolder, symbol Device:C_Small
- removed D1, D2: BLUE, LED_SMD:LED_0603_1608Metric_Pad1.05x0.95mm_HandSolder, symbol Device:LED
- removed J1: USB_A, Connector_USB:USB_A_Stewart_SS-52100-001_Horizontal, symbol 2021_Rev1-rescue:USB_A-Connector
- removed R1, R2: 27, Resistor_SMD:R_0603_1608Metric_Pad0.98x0.95mm_HandSolder, symbol Device:R
- removed R4: 510, Resistor_SMD:R_0603_1608Metric_Pad0.98x0.95mm_HandSolder, symbol Device:R
- removed R5, R6: 330, Resistor_SMD:R_0603_1608Metric_Pad0.98x0.95mm_HandSolder, symbol Device:R
- removed U3: OKI, MRDT_Devices:OKI_Horizontal, symbol MRDT_Devices:OKI
- removed U4: FT230XS, Package_SO:SSOP-16_3.9x4.9mm_P0.635mm, symbol Interface_USB:FT230XS
Connections:
- net labels removed: +5V, KBoard_RX, KBoard_TX
- wire segments 227 -> 151
- no-connect marks 68 -> 69
