File: Hardware/EquipmentServicingPanel_Hardware_2023_Rev1.kicad_pcb (KiCad board)
At the start: 2 copper layers, 42 parts, among them U1 Raspberry_Pi, U2 OKI, U3 TSR_1-2450

Commit message: Made layout
Parts:
- added G***: LOGO, MRDT_Silkscreens:Sean_Duda_Signature_41.0mmx30.7mm, F.Cu at (165.6, 115.3)
- added G***: LOGO, MRDT_Silkscreens:z_sig_Grant_Brinker_25mmx6, F.Cu at (140.7, 116.3)
- added G***: LOGO, MRDT_Silkscreens:0_MRDT_Logo_10mm, F.Cu at (128.0, 103.1)
- C1, C2: footprint Capacitor_SMD:C_0201_0603Metric_Pad0.64x0.40mm_HandSolder -> Capacitor_SMD:C_0603_1608Metric_Pad1.08x0.95mm_HandSolder
- Conn10, Conn11, Conn12, Conn13, Conn15, Conn17, Conn8, Conn9: footprint MRDT_Connectors:MOLEX_SL_02_Horizontal -> MRDT_Connectors:MOLEX_SL_02_Vertical
- D1, D2, D3, D4, D5, D6, D7: footprint LED_SMD:LED_0201_0603Metric_Pad0.64x0.40mm_HandSolder -> LED_SMD:LED_0603_1608Metric_Pad1.05x0.95mm_HandSolder
- moved C1 104.7 mm to (95.5, 128.8)
- moved U1 85.5 mm to (171.7, 96.8), turned to 90 degrees
- moved C4 80.9 mm to (108.7, 124.5)
- moved V3 78.1 mm to (86.4, 91.4), turned to -90 degrees
- moved U2 76.7 mm to (94.6, 126.4), turned to 180 degrees
- moved Conn15 75.1 mm to (100.6, 108.3)
- moved Conn2 72.6 mm to (158.8, 132.7), turned to 180 degrees
- moved Conn3 72.2 mm to (168.3, 132.7), turned to 180 degrees
- moved Conn1 72.2 mm to (104.8, 132.7)
- moved Conn8 57.6 mm to (120.7, 124.3), turned to 180 degrees
- moved C3 57.2 mm to (102.9, 124.5), turned to 180 degrees
- moved Conn10 54.1 mm to (139.7, 124.3), turned to 180 degrees
- moved Conn9 53.9 mm to (130.2, 124.3), turned to 180 degrees
- moved V2 53.9 mm to (180.3, 146.1), turned to 90 degrees
- moved Conn16 48.8 mm to (110.2, 102.6)
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Connections:
- U1 pad 1: Net-(U1-Pad1) -> unconnected-(U1-Pad1)
- U1 pad 10: Net-(U1-Pad10) -> unconnected-(U1-Pad10)
- U1 pad 12: Net-(U1-Pad12) -> unconnected-(U1-Pad12)
- U1 pad 13: Net-(U1-Pad13) -> unconnected-(U1-Pad13)
- U1 pad 15: Net-(U1-Pad15) -> unconnected-(U1-Pad15)
- U1 pad 16: Net-(U1-Pad16) -> unconnected-(U1-Pad16)
- U1 pad 17: Net-(U1-Pad17) -> unconnected-(U1-Pad17)
- U1 pad 19: Net-(U1-Pad19) -> unconnected-(U1-Pad19)
- U1 pad 21: Net-(U1-Pad21) -> unconnected-(U1-Pad21)
- U1 pad 22: Net-(U1-Pad22) -> unconnected-(U1-Pad22)
- U1 pad 23: Net-(U1-Pad23) -> unconnected-(U1-Pad23)
- U1 pad 24: Net-(U1-Pad24) -> unconnected-(U1-Pad24)
- U1 pad 26: Net-(U1-Pad26) -> unconnected-(U1-Pad26)
- U1 pad 27: Net-(U1-Pad27) -> unconnected-(U1-Pad27)
- U1 pad 28: Net-(U1-Pad28) -> unconnected-(U1-Pad28)
- U1 pad 29: Net-(U1-Pad29) -> unconnected-(U1-Pad29)
- U1 pad 3: Net-(U1-Pad3) -> unconnected-(U1-Pad3)
- U1 pad 36: Net-(U1-Pad36) -> unconnected-(U1-Pad36)
- U1 pad 38: Net-(U1-Pad38) -> unconnected-(U1-Pad38)
- U1 pad 4: Net-(U1-Pad4) -> unconnected-(U1-Pad4)
- U1 pad 40: Net-(U1-Pad40) -> unconnected-(U1-Pad40)
- U1 pad 5: Net-(U1-Pad5) -> unconnected-(U1-Pad5)
- U1 pad 7: Net-(U1-Pad7) -> unconnected-(U1-Pad7)
- U1 pad 8: Net-(U1-Pad8) -> unconnected-(U1-Pad8)
Routing:
- net +12V: track 0.00 -> 130.2 mm
- net +5V: track 0.00 -> 113.8 mm
- net ELEV_MINUS: track 0.00 -> 74.2 mm, vias 0 -> 2
- net ELEV_PLUS: track 0.00 -> 73.6 mm, vias 0 -> 1
- net AZI_MINUS: track 0.00 -> 73.5 mm, vias 0 -> 1
- net +3V3: track 0.00 -> 65.5 mm, vias 0 -> 2
- net ELEV_CNTRL: track 0.00 -> 48.8 mm, vias 0 -> 2
- net AZI_CNTRL: track 0.00 -> 44.1 mm
- net AZI_PLUS: track 0.00 -> 40.0 mm, vias 0 -> 1
- net Net-(D4-Pad2): track 0.00 -> 2.02 mm
- net Net-(D3-Pad2): track 0.00 -> 2.02 mm
- net Net-(D2-Pad2): track 0.00 -> 2.02 mm
- net Net-(D1-Pad2): track 0.00 -> 2.02 mm
- net Net-(D7-Pad2): track 0.00 -> 1.78 mm
- net Net-(D5-Pad2): track 0.00 -> 1.77 mm
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- added copper zone on F.Cu, net +12V
- added copper zone on B.Cu, net GND
- added copper zone on F.Cu, net GND
Other:
- board outline added: 94 x 54.6 mm
- net class Default removed
- board text added: "12V"
- board text added: "3.3V"
- board text added: "5V"
- board text added: "AZI CTRL"
- board text added: "Ammo Crate LED"
- board text added: "Azimuth"
- board text added: "ELEV CTRL"
- board text added: "Elevation"
- board text added: "Equipment Servicing Panel Board, Rev 1 Mars Rover Design Team Missouri S&T, 2023 Grant Brinker, Sean Duda"
- board text added: "Hex Bolt LED"
- board text added: "Push Buttons"
- board text added: "Switches"
