File: Hardware/Hardware_2024/Hardware_2024.kicad_pcb (KiCad board)
At the start: 2 copper layers, 127 x 57.9 mm, 51 parts, among them U1 Raspberry_Pi, U2 SHHD003A0A, U3 MCP3008

Commit message: Updated with changes
Parts:
- removed C3: 100uF, Capacitor_THT:CP_Radial_D6.3mm_P2.50mm
- removed C4: 220uF, Capacitor_THT:CP_Radial_D6.3mm_P2.50mm
- removed Conn10, Conn11, Conn12, Conn13, Conn18, Conn19, Conn20, Conn21, Conn22, Conn23, Conn24, Conn25, Conn4, Conn5, Conn6, Conn7, Conn8, Conn9: Molex_SL_02, MRDT_Connectors:MOLEX_SL_02_Vertical
- removed Conn26: Molex_SL_03, MRDT_Connectors:MOLEX_SL_03_Vertical
- removed D1, D2, D3, D4: LED, LED_SMD:LED_0603_1608Metric_Pad1.05x0.95mm_HandSolder
- removed R1, R2, R3, R4: 100, Resistor_SMD:R_0603_1608Metric_Pad0.98x0.95mm_HandSolder
- removed U3: MCP3008, Package_DIP:DIP-16_W7.62mm
- Conn1: footprint MRDT_Connectors:Square_Anderson_2_H_Stacked -> MRDT_Connectors:Square_Anderson_2_H_Side_By_Side
- U1: footprint MRDT_Shields:RASPBERRY_PI_HEADERS -> MRDT_Shields:RaspberryPi_THT_BOTTOM
- U2: footprint SHHD003A04A41:SHHD003A0A-SRZ -> MRDT_Devices:SHHD003A0A41Z_Through_Hole
- moved V4 128.6 mm to (0.25, 8.10), turned to 0 degrees
- moved V3 97.4 mm to (0.25, 8.10), turned to 0 degrees
- moved U1 85.1 mm to (110.9, 112.9), turned to 0 degrees
- moved V2 66.3 mm to (119.1, 104.7), turned to 180 degrees
- moved V1 66.2 mm to (118.9, 67.5), turned to 90 degrees
- moved Conn2 62.9 mm to (204.0, 74.4)
- moved Conn3 51.2 mm to (196.5, 74.4)
- moved Conn14 45.3 mm to (189.0, 74.4)
- moved Conn1 43.5 mm to (127.8, 90.6)
- moved U2 38.6 mm to (124.6, 85.1)
- moved Conn15 34.3 mm to (181.5, 74.4)
- moved C1 34.2 mm to (120.7, 82.1), turned to 180 degrees
- moved Conn16 29.8 mm to (174.0, 74.4)
- moved Conn17 29.6 mm to (166.5, 74.4)
- moved C2 26.3 mm to (116.2, 82.0), turned to 180 degrees
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Connections:
- net +3.3V renamed +3V3
- U1 pad 10: LED2 -> unconnected-(U1-GP_15-Pad10)
- U1 pad 11: Sw4 -> unconnected-(U1-GP_17-Pad11)
- U1 pad 12: LED3 -> unconnected-(U1-GP_18-Pad12)
- U1 pad 13: Sw5 -> unconnected-(U1-GP_27-Pad13)
- U1 pad 15: Sw6 -> unconnected-(U1-GP_22-Pad15)
- U1 pad 16: LED4 -> unconnected-(U1-GP_23-Pad16)
- U1 pad 18: LED5 -> unconnected-(U1-GP_24-Pad18)
- U1 pad 19: DIN -> unconnected-(U1-GP_10-Pad19)
- U1 pad 21: DOUT -> unconnected-(U1-GP_9-Pad21)
- U1 pad 22: LED6 -> unconnected-(U1-GP_25-Pad22)
- U1 pad 23: CLK -> unconnected-(U1-GP_11-Pad23)
- U1 pad 24: CS -> unconnected-(U1-GP_8-Pad24)
- U1 pad 26: LED7 -> unconnected-(U1-GP_7-Pad26)
- U1 pad 27: Sw7 -> unconnected-(U1-GP_0-Pad27)
- U1 pad 28: LED8 -> unconnected-(U1-GP_1-Pad28)
- U1 pad 3: Sw1 -> unconnected-(U1-GP_2-Pad3)
- U1 pad 36: LED9 -> unconnected-(U1-GP_16-Pad36)
- U1 pad 38: Button2 -> unconnected-(U1-GP_20-Pad38)
- U1 pad 40: Button1 -> unconnected-(U1-GP_21-Pad40)
- U1 pad 5: Sw2 -> unconnected-(U1-GP_3-Pad5)
- U1 pad 7: Sw3 -> unconnected-(U1-GP_4-Pad7)
- U1 pad 8: LED1 -> unconnected-(U1-GP_14-Pad8)
Routing:
- net +3V3: track 200.9 -> 90.6 mm, vias 1 -> 0
- net LED1: track 108.2 -> 0.00 mm, vias 4 -> 0
- net Sw1: track 100.6 -> 0.00 mm, vias 2 -> 0
- net LED2: track 98.6 -> 0.00 mm, vias 4 -> 0
- net Sw2: track 92.9 -> 0.00 mm, vias 2 -> 0
- net Button1: track 91.3 -> 0.00 mm, vias 3 -> 0
- net LED3: track 88.2 -> 0.00 mm, vias 2 -> 0
- net Sw3: track 87.3 -> 0.00 mm, vias 2 -> 0
- net LED5: track 87.2 -> 0.00 mm, vias 1 -> 0
- net Sw4: track 85.7 -> 0.00 mm, vias 2 -> 0
- net LED4: track 82.0 -> 0.00 mm, vias 2 -> 0
- net Sw5: track 79.9 -> 0.00 mm, vias 2 -> 0
- net Button2: track 78.3 -> 0.00 mm, vias 2 -> 0
- net Sw7: track 75.4 -> 0.00 mm, vias 3 -> 0
- net LED6: track 73.7 -> 0.00 mm, vias 4 -> 0
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- removed copper zone on F.Cu, net +12V
Other:
- board size 127 x 57.9 mm -> 106.7 x 53.5 mm
- board text added: "12V"
- board text added: "3V3"
- board text added: "5V"
- board text added: "Azimuth +"
- board text added: "Azimuth -"
- board text added: "Azimuth Control"
- board text added: "Elevation +"
- board text added: "Elevation -"
- board text added: "Elevation Control"
- board text added: "Equipment Servicing Breakout Mars Rover Design Team Missouri S&T, 2024 Natasha Cox"
- board text removed: "1"
- board text removed: "2"
- board text removed: "3"
- board text removed: "4"
- board text removed: "5"
- board text removed: "6"
- board text removed: "7"
- board text removed: "8"
- board text removed: "9"
- board text removed: "Azi +"
- board text removed: "Azi -"
- board text removed: "Azi Ctrl"
- board text removed: "Button1"
- board text removed: "Button2"
- board text removed: "Buttons"
- board text removed: "Elev +"
- board text removed: "Elev -"
- board text removed: "Elev Ctrl"
- board text removed: "Equipment Servicing Panel, Rev1 Mars Rover Design Team Missouri S&T, 2024 Natasha Cox"
- board text removed: "Joystick"
- board text removed: "LEDs"
- board text removed: "Switches"
- board text removed: "Voltmeter"
